File: Design/PCB/PCB.kicad_pcb (KiCad board)
At the start: 4 copper layers, 130.9 x 70.5 mm, 101 parts, among them J11 SWD, J12 BLE PROG, J13 RGB_LED, J14 ENABLE, J15 CAN, J6 BAL_BATT, SW1 NRST, SW2 BOOT0, T1 TestPoint, T10 TestPoint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

Commit message: Added final pcb design and manufacturing files
Parts:
- added kibuzzard-65C18164: G***, kibuzzard-65C18164, F.Cu at (126.0, 65.2)
- added kibuzzard-65C181B2: G***, kibuzzard-65C181B2, F.Cu at (113.5, 73.5)
- added kibuzzard-65C181EB: G***, kibuzzard-65C181EB, F.Cu at (137.5, 45.8)
- added kibuzzard-65C18390: G***, kibuzzard-65C18390, F.Cu at (154.0, 32.8)
- added kibuzzard-65C183BF: G***, kibuzzard-65C183BF, F.Cu at (91.5, 50.5)
- added kibuzzard-65C185CB: G***, kibuzzard-65C185CB, B.Cu at (86.0, 50.8)
- added kibuzzard-65C185F9: G***, kibuzzard-65C185F9, F.Cu at (87.2, 70.2)
- added kibuzzard-65C187BD: G***, kibuzzard-65C187BD, F.Cu at (86.0, 60.0)
- added kibuzzard-65C18803: G***, kibuzzard-65C18803, B.Cu at (119.5, 45.8)
- added kibuzzard-65C1883A: G***, kibuzzard-65C1883A, B.Cu at (112.5, 45.8)
- added kibuzzard-65C18854: G***, kibuzzard-65C18854, B.Cu at (104.5, 45.8)
- moved D7 4.77 mm to (110.8, 80.2), turned to 45 degrees
- moved D10 0.50 mm to (108.5, 46.8)
Routing:
- net +3.3V: track 45.5 -> 48.7 mm, vias 25 -> 26
- net GND: track 90.9 -> 88.8 mm, vias 86 -> 89
- net /PWM: track 20.9 -> 19.6 mm
- net unconnected-(U2-SW-Pad4): vias 0 -> 4
- net unconnected-(U1-SW-Pad4): vias 0 -> 4
- added copper zone on B.Cu, net unconnected-(U1-SW-Pad4)
- added copper zone on F.Cu, net unconnected-(U1-SW-Pad4)
- added copper zone on B.Cu, net unconnected-(U2-SW-Pad4)
- added copper zone on F.Cu, net unconnected-(U2-SW-Pad4)
Other:
- board text added: "SWCLK"
- board text added: "SWIO"
- board text added: "SWO"
- board text removed: "A. Loehr"
- board text removed: "Balance Controller"
- board text removed: "RGB"
- board text removed: "Rev. A"
