File: Hardware/Balance_Controller/Balance_Controller.kicad_pcb (KiCad board)
At the start: 4 copper layers, 130.9 x 70.5 mm, 112 parts, among them J11 SWD, J12 BLE PROG, J13 RGB_LED, J14 ENABLE, J15 CAN, J6 BAL_BATT, SW1 NRST, SW2 BOOT0, T1 TestPoint, T10 TestPoint, T11 TestPoint, T2 TestPoint, T3 TestPoint, T4 TestPoint, T6 TestPoint, T7 TestPoint, U1 MPM3610GQV-P, U2 MPM3610GQV-P, U3 TPS2116DRLR, U4 MCP111T-195I/LB, U5 STM32F412CGU6, U6 RN4871-I/RM140, U7 TJA1051TK-3, U8 MPU-6050, Y1 NX3225SA-16.000

Commit message: 17 revise balance controller pcb (#18)
* Added LED board progress

* Updated schematic and routing

* Created updated BOM and manufacturing files

* Updated XT60 PN and added render
Parts:
- removed BATT BALANCE: BAL_CHRG, Connector_JST:JST_XH_B7B-XH-A_1x07_P2.50mm_Vertical
- removed the C12 at (141.5, 34.8)
- removed the C13 at (141.5, 40.0)
- removed the C14 at (147.5, 40.0)
- removed the C18 at (153.5, 26.2)
- removed the D7 at (110.8, 80.2)
- removed the D8 at (138.5, 26.2)
- removed the J11 at (112.8, 77.8)
- removed the J12 at (153.8, 36.7)
- removed the R14 at (138.6, 28.5)
- removed the U3 at (144.5, 38.2)
- removed the U4 at (144.5, 34.8)
- removed U6: RN4871-I/RM140, RN4871-I/RM140:RN4871_MCH
- removed kibuzzard-65C18164: G***, kibuzzard-65C18164
- removed kibuzzard-65C181B2: G***, kibuzzard-65C181B2
- removed kibuzzard-65C18390: G***, kibuzzard-65C18390
- removed kibuzzard-65C185F9: G***, kibuzzard-65C185F9
- added D10: RED, LED_SMD:LED_0805_2012Metric, F.Cu at (137.8, 49.0)
- added D11: VESD03A2-03G-G3-08, Package_TO_SOT_SMD:SOT-323_SC-70, B.Cu at (149.0, 30.2)
- added D12: SC1533-01FTG, Diode_SMD:D_SOD-323, B.Cu at (142.5, 30.2)
- added D6: ESDALC6V1W5, ESDALC6V1W5:SOT65P210X110-5N, F.Cu at (141.8, 43.5)
- added J1: HC-05, Connector_PinSocket_2.54mm:PinSocket_1x06_P2.54mm_Vertical, F.Cu at (140.0, 26.5)
- added J10: BAL_BATT_A, Connector_JST:JST_XH_B4B-XH-A_1x04_P2.50mm_Vertical, F.Cu at (82.2, 54.8)
- added J6: SWD, Connector_PinHeader_1.27mm:PinHeader_2x05_P1.27mm_Vertical_SMD, F.Cu at (141.8, 37.2)
- added R12: 15, Resistor_SMD:R_0603_1608Metric, F.Cu at (131.0, 43.0)
- added kibuzzard-1: G***, kibuzzard-65EC859F, F.Cu at (146.5, 23.2)
- added kibuzzard-2: G***, kibuzzard-65EE22FE, F.Cu at (141.8, 32.5)
- added kibuzzard-6: G***, kibuzzard-65EE0D80, F.Cu at (113.3, 69.8)
- added kibuzzard-65EE6C62: G***, kibuzzard-65EE6C62, F.Cu at (63.8, 46.2)
- added kibuzzard-65EE6C92: G***, kibuzzard-65EE6C92, F.Cu at (70.2, 52.5)
- added kibuzzard-65EE6CA7: G***, kibuzzard-65EE6CA7, F.Cu at (55.0, 23.2)
- added kibuzzard-65EE6CAC: G***, kibuzzard-65EE6CAC, F.Cu at (55.0, 35.8)
- added kibuzzard-7: G***, kibuzzard-65EBE841, F.Cu at (87.2, 70.2)
- D4: value REGEN_BYPASS -> SC1533-01FTG; footprint SBM3060VDC-AU_R2_006A1:SBM3060VDCAU_R2_006A1 -> Diode_SMD:D_SOD-323
- D9: value SC1533-01FTG -> GRN; footprint Diode_SMD:D_SOD-323 -> LED_SMD:LED_0805_2012Metric
- J15: renamed from J6; value BAL_BATT -> BAL_BATT_B
- R11: value 4.7k -> 220
- T1, T4: footprint RCU-0C:TP+195X110 -> RCT-0C:RCT-0C
- T2: renamed from T3; footprint RCU-0C:TP+195X110 -> RCT-0C:RCT-0C
- T3: renamed from T2; footprint RCU-0C:TP+195X110 -> RCT-0C:RCT-0C
- U3: renamed from U5; footprint Package_DFN_QFN:QFN-48-1EP_7x7mm_P0.5mm_EP5.6x5.6mm -> STM32F412:QFN-48-1EP_7x7mm_P0.5mm_EP5.6x5.6mm
- U5: renamed from U8; footprint Sensor_Motion:InvenSense_QFN-24_4x4mm_P0.5mm -> MPU6050:InvenSense_QFN-24_4x4mm_P0.5mm
- moved D4 82.3 mm to (147.0, 34.0)
- moved D9 19.9 mm to (134.8, 49.0), turned to 90 degrees
- moved SW1 19.8 mm to (152.2, 35.8)
- moved kibuzzard-3 19.8 mm to (152.2, 32.5)
- moved R11 17.6 mm to (131.0, 41.0), turned to 0 degrees
- moved J2 12.5 mm to (55.0, 40.5)
- moved J8 10.0 mm to (55.0, 28.0)
- moved D5 6.95 mm to (49.2, 28.0)
- moved SW2 5.27 mm to (117.1, 73.8)
- moved C9 0.25 mm to (118.2, 49.0)
- renumbered C4 to C1, C16 to C10, C15 to C11, C27 to C12, C17 to C13, C25 to C14, C28 to C15, C20 to C16, C26 to C17, C8 to C18, C1 to C2, C10 to C20, C11 to C21, C31 to C22, C32 to C23, C30 to C24, C24 to C25, C23 to C26, C29 to C27, C22 to C28, C5 to C3, C6 to C4, C2 to C5, C3 to C6, C9 to C8, C21 to C9, D5 to D1, D11 to D13, D10 to D14, D1 to D3, D6 to D5, D12 to D7, D3 to D8, H2 to H1, H3 to H2, H1 to H3, BATT- to J11, J14 to J12, J15 to J14, VESC- to J2, COM_SW to J3, LOAD_SW to J4, CHRG_SW to J5, CHARGE to J7, VESC+ to J8, BATT+ to J9, R10 to R1, R7 to R10, R17 to R13, R18 to R14, R12 to R15, R13 to R16, R16 to R17, R15 to R18, R3 to R2, R9 to R3, R1 to R4, R6 to R5, R5 to R6, R4 to R7, R2 to R8, R8 to R9, T11 to T5, T10 to T6, T6 to T7, T7 to T8, U2 to U1, U1 to U2, U7 to U4, kibuzzard-65C18854 to kibuzzard-10, kibuzzard-65C185CB to kibuzzard-11, kibuzzard-65C181EB to kibuzzard-3, kibuzzard-65C183BF to kibuzzard-4, kibuzzard-65C187BD to kibuzzard-5, kibuzzard-65C18803 to kibuzzard-8, kibuzzard-65C1883A to kibuzzard-9
Connections:
- D4 pad 1: +12V -> GND
- D4 pad 2: /VBAT -> +3.3V
- D9 pad 2: /VPROG -> Net-(D9-A)
- R11 pad 1: /BLE_NRST -> /LED_R
- R11 pad 2: /VBLE -> Net-(D10-A)
- U3 pad 17: unconnected-(U5-PA7-Pad17) -> /LED_G
- U3 pad 18: unconnected-(U5-PB0-Pad18) -> /LED_R
Routing:
- net /SWIO: track 22.3 -> 60.8 mm, vias 1 -> 2
- net /SWCLK: track 18.2 -> 49.8 mm, vias 1 -> 2
- net /VBLE: track 27.5 -> 0.00 mm
- net /SW0: track 17.8 -> 45.1 mm, vias 1 -> 2
- net /NRST: track 21.9 -> 48.6 mm, vias 3 -> 4
- net /LED_R: track 0.00 -> 16.1 mm
- net /BLE_ON_LED_K: track 16.0 -> 0.00 mm, vias 2 -> 0
- net /BLE_MODE: track 14.8 -> 0.00 mm, vias 1 -> 0
- net /LED_G: track 0.00 -> 14.3 mm
- net Net-(D10-A): track 0.00 -> 10.8 mm
- net /UART_RX: track 51.3 -> 40.9 mm
- net /VPROG: track 9.63 -> 0.00 mm
- net +5V: track 15.7 -> 24.5 mm
- net /UART_TX: track 51.7 -> 44.1 mm
- net Net-(D9-A): track 0.00 -> 6.82 mm
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- removed copper zone on F.Cu, net /BLE_NRST
- removed copper zone on F.Cu, net /VBLE
Other:
- board text removed: "GND"
- board text removed: "MODE"
- board text removed: "RX"
- board text removed: "SWCLK"
- board text removed: "SWIO"
- board text removed: "SWO"
- board text removed: "TX"
