File: Hardware/Balance_Controller/Balance_Controller.kicad_sch (KiCad schematic)
At the start: 101 parts, among them J1 COM_SW, J10 VESC-, J11 SWD, J12 BLE PROG, J13 RGB_LED, J14 ENABLE, J15 CAN, J2 CHRG_SW, J3 LOAD_SW, J4 BATT+, J5 BATT-, J6 BAL_BATT, J7 BAL_CHRG, J8 CHARGE, J9 VESC+, SW1 NRST, SW2 BOOT0, T1 TestPoint, T10 TestPoint, T11 TestPoint, T2 TestPoint, T3 TestPoint, T4 TestPoint, T6 TestPoint, T7 TestPoint, U1 MPM3610GQV-P, U2 MPM3610GQV-P, U3 TPS2116DRLR, U4 MCP111T-195I/LB, U5 STM32F412CGU6, U6 RN4871-I/RM140, U7 TJA1051TK-3, U8 MPU-6050, Y1 NX3225SA-16.000

Commit message: 17 revise balance controller pcb (#18)
* Added LED board progress

* Updated schematic and routing

* Created updated BOM and manufacturing files

* Updated XT60 PN and added render
Parts:
- removed C12: 100n, Capacitor_SMD:C_0603_1608Metric, symbol Device:C
- removed C13, C14: 1u, Capacitor_SMD:C_0805_2012Metric, symbol Device:C
- removed C18: 10u, Capacitor_SMD:C_1206_3216Metric, symbol Device:C
- removed D4: REGEN_BYPASS, SBM3060VDC-AU_R2_006A1:SBM3060VDCAU_R2_006A1, symbol SBM3060VDC-AU_R2_006A1:SBM3060VDC-AU_R2_006A1
- removed D7, D9: SC1533-01FTG, Diode_SMD:D_SOD-323, symbol Device:D_TVS
- removed D8: BLUE, LED_SMD:LED_0805_2012Metric, symbol Device:LED
- removed J11: SWD, Connector_PinHeader_1.27mm:PinHeader_1x05_P1.27mm_Vertical, symbol Connector:Conn_01x05_Pin
- removed J12: BLE PROG, Connector_PinHeader_1.27mm:PinHeader_1x05_P1.27mm_Vertical, symbol Connector:Conn_01x05_Pin
- removed J7: BAL_CHRG, Connector_JST:JST_XH_B7B-XH-A_1x07_P2.50mm_Vertical, symbol Connector_Generic:Conn_01x07
- removed R14: 300, Resistor_SMD:R_0603_1608Metric, symbol Device:R
- removed U3: TPS2116DRLR, TPS2116DRLR:SOTFL50P160X60-8N, symbol TPS2116DRLR:TPS2116DRLR
- removed U4: MCP111T-195I/LB, MCP111T-195I/LB:SOT65P210X110-3N, symbol MCP111T-195I_LB:MCP111T-195I_LB
- removed U6: RN4871-I/RM140, RN4871-I/RM140:RN4871_MCH, symbol RN4871-I/RM140:RN4871-I_RM140
- added D10: RED, LED_SMD:LED_0805_2012Metric, symbol Device:LED
- added D11: VESD03A2-03G-G3-08, Package_TO_SOT_SMD:SOT-323_SC-70, symbol VESD: VESD03A2-03G-G3-08
- added D12, D4: SC1533-01FTG, Diode_SMD:D_SOD-323, symbol Device:D_TVS
- added D6: ESDALC6V1W5, ESDALC6V1W5:SOT65P210X110-5N, symbol ESDALC6V1W5:ESDALC6V1W5
- added D9: GRN, LED_SMD:LED_0805_2012Metric, symbol Device:LED
- added J1: HC-05, Connector_PinSocket_2.54mm:PinSocket_1x06_P2.54mm_Vertical, symbol Connector:Conn_01x06_Socket
- added J10: BAL_BATT_A, Connector_JST:JST_XH_B4B-XH-A_1x04_P2.50mm_Vertical, symbol Connector_Generic:Conn_01x04
- added J6: SWD, Connector_PinHeader_1.27mm:PinHeader_2x05_P1.27mm_Vertical_SMD, symbol Connector_Generic:Conn_02x05_Odd_Even
- added R12: 15, Resistor_SMD:R_0603_1608Metric, symbol Device:R
- C1: renamed from C4; MFG (none) -> Murata; MPN (none) -> GRM32ER71E226KE15L; PN GRM32ER71E226KE15L -> (none)
- C10: renamed from C16; MFG (none) -> Murata; MPN (none) -> GRM21BR71C105KA01K; PN GRM21BR71C105KA01K -> (none)
- C11: renamed from C15; MFG (none) -> Murata; MPN (none) -> GRM21BR71C105KA01K; PN GRM21BR71C105KA01K -> (none)
- C12: renamed from C27; MFG (none) -> Murata; MPN (none) -> GCJ188R71C473KA01D; PN GCJ188R71C473KA01D -> (none)
- C13: renamed from C17; MFG (none) -> Murata; MPN (none) -> GRM188R72A104KA35J; PN GRM188R72A104KA35J -> (none)
- C14: renamed from C25; MFG (none) -> Murata; MPN (none) -> GCM1885C1H101JA16J; PN GCM1885C1H101JA16J -> (none)
- C15: renamed from C28; MFG (none) -> Murata; MPN (none) -> GCM1885C1H101JA16J; PN GCM1885C1H101JA16J -> (none)
- C16: renamed from C20; MFG (none) -> Murata; MPN (none) -> GRM1885C2A6R0DA01D; PN GRM1885C2A6R0DA01D -> (none)
- C17: renamed from C26; MFG (none) -> Murata; MPN (none) -> GRM188R72A104KA35J; PN GRM188R72A104KA35J -> (none)
- C18: renamed from C8; MFG (none) -> Murata; MPN (none) -> GRM188R72A104KA35J; PN GRM188R72A104KA35J -> (none)
- C19: MFG (none) -> Murata; MPN (none) -> GRM1885C2A6R0DA01D; PN GRM1885C2A6R0DA01D -> (none)
- C2: renamed from C1; MFG (none) -> Murata; MPN (none) -> GRM32ER71E226KE15L; PN GRM32ER71E226KE15L -> (none)
- C20: renamed from C10; MFG (none) -> Murata; MPN (none) -> GRM188R72A104KA35J; PN GRM188R72A104KA35J -> (none)
- C21: renamed from C11; MFG (none) -> Murata; MPN (none) -> GRM188R72A104KA35J; PN GRM188R72A104KA35J -> (none)
- C22: renamed from C31; MFG (none) -> Murata; MPN (none) -> GRM31CR71E106MA12L; PN GRM31CR71E106MA12L -> (none)
- C23: renamed from C32; MFG (none) -> Murata; MPN (none) -> GCJ188R71C473KA01D; PN GCJ188R71C473KA01D -> (none)
- C24: renamed from C30; MFG (none) -> Murata; MPN (none) -> GRT1885C1H222JA02D; PN GRT1885C1H222JA02D -> (none)
- C25: renamed from C24; MFG (none) -> Murata; MPN (none) -> GRM188R72A104KA35J; PN GRM188R72A104KA35J -> (none)
- C26: renamed from C23; MFG (none) -> Murata; MPN (none) -> GRM1885C1H103JA01J; PN GRM1885C1H103JA01J -> (none)
- C27: renamed from C29; MFG (none) -> Murata; MPN (none) -> GRM188R72A104KA35J; PN GRM188R72A104KA35J -> (none)
- C28: renamed from C22; MFG (none) -> Murata; MPN (none) -> GRM188R72A104KA35J; PN GRM188R72A104KA35J -> (none)
- C3: renamed from C5; MFG (none) -> Murata; MPN (none) -> GRM32ER71E226KE15L; PN GRM32ER71E226KE15L -> (none)
- C4: renamed from C6; MFG (none) -> Murata; MPN (none) -> GRM32ER71E226KE15L; PN GRM32ER71E226KE15L -> (none)
- C5: renamed from C2; MFG (none) -> Murata; MPN (none) -> GRM32ER71E226KE15L; PN GRM32ER71E226KE15L -> (none)
- C6: renamed from C3; MFG (none) -> Murata; MPN (none) -> GRM32ER71E226KE15L; PN GRM32ER71E226KE15L -> (none)
- C7: MFG (none) -> Murata; MPN (none) -> GRM31CR71E106MA12L; PN GRM31CR71E106MA12L -> (none)
- C8: renamed from C9; MFG (none) -> Murata; MPN (none) -> GRM188R72A104KA35J; PN GRM188R72A104KA35J -> (none)
- C9: renamed from C21; MFG (none) -> Murata; MPN (none) -> GRM21BZ71E475KE15L; PN GRM21BZ71E475KE15L -> (none)
- D1: renamed from D5; MFG (none) -> Panjit; Manufacturer Panjit -> (none)
- D13: renamed from D11; MFG (none) -> Littelfuse; MPN (none) -> SC1533-01FTG; PN SC1533-01FTG -> (none)
- D14: renamed from D10; MFG (none) -> Littelfuse; MPN (none) -> SC1533-01FTG; PN SC1533-01FTG -> (none)
- D2: MFG (none) -> Wurth Elektronik; MPN (none) -> 150080SS75000; PN 150080SS75000 -> (none)
- D3: renamed from D1; MFG (none) -> Wurth Elektronik; MPN (none) -> 150080SS75000; PN 150080SS75000 -> (none)
- D5: renamed from D6; MFG (none) -> Panjit; Manufacturer Panjit -> (none)
- D7: renamed from D12; MFG (none) -> Diotec; MPN (none) -> NUP2105L
- D8: renamed from D3; MFG (none) -> Panjit; Manufactuer Panjit -> (none)
- F1: MFG (none) -> Keystone Electronics; Manufacturer_Name Keystone Electronics -> (none); Manufacturer_Part_Number 3568 -> (none)
- FB1: MFG (none) -> Murata; MPN (none) -> BLM18KG121TN1D; PN BLM18KG121TN1D -> (none)
- H1: renamed from H2; now left out of the parts list
- H2: renamed from H3; now left out of the parts list
- H3: renamed from H1; now left out of the parts list
- J11: renamed from J5; now left out of the parts list
- J12: renamed from J14; MFG (none) -> JST; MPN (none) -> B2B-PH-K; PN B2B-PH-K -> (none)
- J13: MFG (none) -> JST; MPN (none) -> B2B-PH-K; PN B2B-PH-K -> (none)
- J14: renamed from J15; MFG (none) -> JST; MPN (none) -> B3B-PH-K; PN B3B-PH-K -> (none)
- J15: renamed from J6; value BAL_BATT -> BAL_BATT_B; MFG (none) -> JST; Manufacturer JST -> (none)
- J2: renamed from J10; now left out of the parts list
- J3: renamed from J1; now left out of the parts list
- J4: renamed from J3; now left out of the parts list
- J5: renamed from J2; now left out of the parts list
- J7: renamed from J8; MFG (none) -> AMASS; MPN XT60-F -> XT60PB-F; Manufacturer AMASS -> (none)
- J8: renamed from J9; now left out of the parts list
- J9: renamed from J4; now left out of the parts list
- R1: renamed from R10; MFG (none) -> Panasonic; MPN (none) -> ERJ-PA3F5362V; PN ERJ-PA3F5362V -> (none)
- R10: renamed from R7; MFG (none) -> Vishay; MPN (none) -> CRCW060312K7FKEAHP; PN CRCW060312K7FKEAHP -> (none)
- R11: value 4.7k -> 220; MFG (none) -> Panasonic; MPN (none) -> ERJ-UP3J221V; PN MCT0603MD4701BP500 -> (none)
- R13: renamed from R17; MFG (none) -> Panasonic; MPN (none) -> ERJ-UP3F60R4V; PN ERJ-UP3F60R4V -> (none)
- R14: renamed from R18; MFG (none) -> Panasonic; MPN (none) -> ERJ-UP3F60R4V; PN ERJ-UP3F60R4V -> (none)
- R15: renamed from R12; MFG (none) -> Vishay; MPN (none) -> MCT0603MD4701BP500; PN MCT0603MD4701BP500 -> (none)
- R16: renamed from R13; MFG (none) -> Vishay; MPN (none) -> MCT0603MD4701BP500; PN MCT0603MD4701BP500 -> (none)
- R17: renamed from R16; MFG (none) -> ROHM; MPN (none) -> ESR03EZPJ103; PN ESR03EZPJ103 -> (none)
- R18: renamed from R15; MFG (none) -> ROHM; MPN (none) -> ESR03EZPJ103; PN ESR03EZPJ103 -> (none)
- R2: renamed from R3; MFG (none) -> Panasonic; MPN (none) -> ERJ-UP3F1003V; PN ERJ-UP3F1003V -> (none)
- R3: renamed from R9; MFG (none) -> Panasonic; MPN (none) -> ERJ-UP3J393V; PN ERJ-UP3J393V -> (none)
- R4: renamed from R1; MFG (none) -> Panasonic; MPN (none) -> ERJ-UP3F1003V; PN ERJ-UP3F1003V -> (none)
- R5: renamed from R6; MFG (none) -> Panasonic; MPN (none) -> ERJ-PA3F5230V; PN ERJ-PA3F5230V -> (none)
- R6: renamed from R5; MFG (none) -> Panasonic; MPN (none) -> ERJ-UP3J221V; PN ERJ-UP3J221V -> (none)
- R7: renamed from R4; MFG (none) -> Panasonic; MPN (none) -> ERJ-PB3D3402V; PN ERJ-PB3D3402V -> (none)
- R8: renamed from R2; MFG (none) -> Vishay; MPN (none) -> RCS060340K2FKEA; PN RCS060340K2FKEA -> (none)
- R9: renamed from R8; MFG (none) -> Panasonic; MPN (none) -> ERJ-PA3F6491V; PN ERJ-PA3F6491V -> (none)
- SW1: MFG (none) -> C&K; MPN (none) -> PTS815 SJG 250 SMTR LFS; Manufacturer_Name C & K COMPONENTS -> (none); Manufacturer_Part_Number PTS815 SJG 250 SMTR LFS -> (none)
- SW2: MFG (none) -> C&K; MPN (none) -> AYZ0102AURLC; PN AYZ0102AURLC -> (none)
- T1: footprint RCU-0C:TP+195X110 -> RCT-0C:RCT-0C; MFG (none) -> TE; MPN RCU-0C -> RCT-0C; Manufacturer TE Connectivity -> (none)
- T2: renamed from T3; footprint RCU-0C:TP+195X110 -> RCT-0C:RCT-0C; MFG (none) -> TE; MPN (none) -> RCT-0C; PN RCU-0C -> (none)
- T3: renamed from T2; footprint RCU-0C:TP+195X110 -> RCT-0C:RCT-0C; MFG (none) -> TE; MPN (none) -> RCT-0C; PN RCU-0C -> (none)
- T4: footprint RCU-0C:TP+195X110 -> RCT-0C:RCT-0C; MFG (none) -> TE; MPN (none) -> RCU-0C; PN RCU-0C -> (none)
- T5: renamed from T11; MFG (none) -> TE; MPN (none) -> RCU-0C; PN RCU-0C -> (none)
- T6: renamed from T10; MFG (none) -> TE; MPN (none) -> RCU-0C; PN RCU-0C -> (none)
- T7: renamed from T6; MFG (none) -> TE; MPN (none) -> RCU-0C; PN RCU-0C -> (none)
- T8: renamed from T7; MFG (none) -> TE; MPN (none) -> RCU-0C; PN RCU-0C -> (none)
- U1: renamed from U2; MFG (none) -> Monolithic Power Systems
- U2: renamed from U1; MFG (none) -> Monolithic Power Systems
- U3: renamed from U5; footprint Package_DFN_QFN:QFN-48-1EP_7x7mm_P0.5mm_EP5.6x5.6mm -> STM32F412:QFN-48-1EP_7x7mm_P0.5mm_EP5.6x5.6mm; MFG (none) -> ST; MPN (none) -> STM32F412CGU6
- U4: renamed from U7; MFG (none) -> NXP; MPN (none) -> TJA1051TK/3,118
- U5: renamed from U8; footprint Sensor_Motion:InvenSense_QFN-24_4x4mm_P0.5mm -> MPU6050:InvenSense_QFN-24_4x4mm_P0.5mm; MFG (none) -> TDK InvenSense
- Y1: MFG (none) -> NDK; MPN (none) -> NX3225SA-16.000M-STD-CRS-2; Part Number NX3225SA-16.000M-STD-CRS-2 -> (none)
Connections:
- net BLE_NRST is gone; now on net LED_R: R11.1
- net +3.3V: now also D4.2 (A2), J6.1 (Pin_1)
- net +5V: now also D12.2 (A2), J1.2 (Pin_2)
- net GND: now also D10.1 (K), D11.3 (GND), D12.1 (A1), D4.1 (A1), D6.2 (GND), D9.1 (K), J1.3 (Pin_3), J6.3 (Pin_3), J6.5 (Pin_5), J6.9 (Pin_9)
- net NRST: now also D6.1 (IO1), J6.10 (Pin_10)
- net SW0: now also D6.5 (IO4), J6.6 (Pin_6)
- net SWCLK: now also D6.4 (IO3), J6.4 (Pin_4)
- net SWIO: now also D6.3 (IO2), J6.2 (Pin_2)
- net UART_RX: now also D11.1 (IO1), J1.4 (Pin_4)
- net UART_TX: now also D11.2 (IO2), J1.5 (Pin_5)
- net LED_G: now reaches U3.17 (PA7)
- net LED_G: now also R12.1
- net LED_R: now reaches U3.18 (PB0)
- net at J15.1 (Pin_1): now also J10.1 (Pin_1)
- net at J15.2 (Pin_2): now also J10.2 (Pin_2)
- net at J15.3 (Pin_3): now also J10.3 (Pin_3)
- net at J15.4 (Pin_4): now also J10.4 (Pin_4)
- net VBLE: no longer names the net of R11.2
- net VBLE: now also D10.2 (A)
- new net: D9.2 (A), R12.2
- no-connect marks 43 -> 34
Other:
- note added: "B"
- note added: "Battery Balance Pass-Thru"
- note added: "J12, J13: JST PHR-2 Terminals: SPH-002T-P0.5L"
- note added: "J14: JST PHR-3 Terminals: SPH-002T-P0.5L"
- note added: "J3-J5 act as e-stop/charge mode select Connect to external SPDT switch (VBAT = COM)"
- note added: "J7: XT60-M"
- note added: "SWD"
- note added: "Status LED's"
- note removed: "Battery Balancer"
- note removed: "J1-J3 act as e-stop/charge mode select Connect to external SPDT switch (VBAT = COM)"
- note removed: "J11: JST PHR-3 Terminals: SPH-002T-P0.5L"
- note removed: "J8: XT60-M"
- note removed: "J9, J10: JST PHR-2 Terminals: SPH-002T-P0.5L"
- note removed: "Power Drop Protection"
- note removed: "Power Mux"
- note removed: "Prevents VPROG (J8) from powering entire +3.3V rail Input 1 takes priority until voltage <1V"
- note removed: "Prog/Debug"
- note removed: "Resets chip once VDD drops below threshold voltage Threshold voltage = 1.95V"
- note removed: "UART BLE Module"
- company: Created By: Austyn Loehr -> (none)
- title: Reaction Wheel Controller -> Balance Controller
- moved on the sheet: C1, C10, C11, C13, C16, C18, C19, C2, C20, C21, C28, C3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
